File: watt-the-mesh.kicad_pcb (KiCad board)
At the start: 2 copper layers, 11 parts, among them U2 TPS61022RWUR

Commit message: minor changes
Parts:
- removed En: TestPoint_Pad_D1.0mm, TestPoint:TestPoint_Pad_D1.0mm
- added REF**: TestPoint_Pad_D1.0mm, TestPoint:TestPoint_Pad_D1.0mm, B.Cu at (110.6, 71.4)
- added U1: nice_nano, PCM_marbastlib-xp-promicroish:nice_nano_AH_USBup_smd, B.Cu at (185.5, 83.0)
- added U3: E22P-915M30S, easyeda:COMM-SMD_22P-P2.54-L38.5-W24.0_E22-400M33S, F.Cu at (152.2, 79.4)
- C3: value C_Small -> 22uf
Connections:
- net /5v renamed +5V
- net /Vbat renamed +BATT
Routing:
- net /Buck_en: track 6.72 -> 1.62 mm, vias 0 -> 1

Commit message: minor schematics changes
Parts:
- U1: footprint PCM_marbastlib-xp-promicroish:nice_nano_AH_USBup_smd -> PCM_marbastlib-xp-promicroish:nice_nano_AH_USBup; moved to F.Cu
- turned U1 to 0 degrees
